Commit message: Setup Project

File: resource/robot.urdf (robot description, URDF)
Before this commit: robot e-puck, 0 links, 0 joints
Links:
- added link base_link
- added link left_wheel
- added link right_wheel
Joints:
- added joint left wheel motor: type continuous, parent base_link, child left_wheel, origin xyz=0 0.026 0, axis 0 1 0
- added joint right wheel motor: type continuous, parent base_link, child right_wheel, origin xyz=0 -0.026 0, axis 0 1 0

Commit message: created robot proto, and make them follow eachothers

File: resource/robot.urdf (robot description, URDF)
Before this commit: robot ri_a1_robot, 3 links, 2 joints
Links:
- removed link left_wheel
- removed link right_wheel
Joints:
- removed joint left wheel motor
- removed joint right wheel motor
